File: discretefpga.sch (EAGLE design)
At the start: 49 parts, among them IC1 74HC595D, IC10 74HC251D, IC11 74HC595D, IC12 74HC595D, IC13 74HC173D, IC3 74HC251D, IC4 74HC125D, IC5 74HC126D, IC6 4066D, IC7 74HC126D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

Commit message: updated schematic
Connections:
- net A_SEL renamed L0_TO_A/L1_TO_A_E0
- net B_SEL renamed U1_TO_B/U0_TO_B_E0
- net C_SEL renamed R0_TO_C/R1_TO_C_E0
- net EW0_SW renamed L0_TO_R0
- net EW1_SW renamed L1_TO_R1
- net LATCHING renamed LATCHING_E0
- net NS0_SW renamed U1_TO_D1
- net NS1_SW renamed U0_TO_D0
- net O0_S0_EN renamed O0_TO_D1
- net O0_S1_EN renamed O0_TO_D0_E0
- net O1_E0_EN renamed O1_TO_R0
- net O1_E1_EN renamed O1_TO_R1_E0
